Commit message: Create tcp_pose property

File: src/maniskill_elirobots/assets/ec63/ec63_description.urdf (robot description, URDF)
Before this commit: robot ec63, 12 links, 11 joints
Links:
- added link claw_tcp_link
Joints:
- added joint claw_tcp_joint: type fixed, parent claw_base, child claw_tcp_link, origin xyz=0 0 0.050 rpy=0 0 0

Commit message: Update EC63 description

File: src/maniskill_elirobots/assets/ec63/ec63_description.urdf (robot description, URDF)
Before this commit: robot ec63, 13 links, 12 joints
Links:
- link claw_finger_1: geometry collision box size=0.005 0.008 0.025; visual box size=0.005 0.008 0.016
- link claw_finger_2: geometry collision box size=0.005 0.008 0.025; visual box size=0.005 0.008 0.016
Joints:
- joint claw_joint: origin xyz=0 0 0 rpy=0 0 0 -> xyz=0 0 0.034 rpy=0 0 0
- joint claw_tcp_joint: origin xyz=0 0 0.050 rpy=0 0 0 -> xyz=0 0 0.109 rpy=0 0 0; parent claw_base -> flan

Commit message: Fix collision meshes

File: src/maniskill_elirobots/assets/ec63/ec63_description.urdf (robot description, URDF)
Before this commit: robot ec63, 13 links, 12 joints
Links:
- link claw_finger_1: geometry collision box size=0.005 0.008 0.041; visual box size=0.005 0.008 0.016
- link claw_finger_2: geometry collision box size=0.005 0.008 0.041; visual box size=0.005 0.008 0.016

Commit message: Update claw definition

File: src/maniskill_elirobots/assets/ec63/ec63_description.urdf (robot description, URDF)
Before this commit: robot ec63, 13 links, 12 joints
Joints:
- joint finger_1_joint: limit lower=0 upper=0.01 effort=10 velocity=0.1 -> lower=0 upper=0.02 effort=10 velocity=0.1; origin xyz=0.02 0 0.042 rpy=0 0 0 -> xyz=0.025 0 0.042 rpy=0 0 0
- joint finger_2_joint: limit lower=0 upper=0.01 effort=10 velocity=0.1 -> lower=0 upper=0.02 effort=10 velocity=0.1; origin xyz=-0.02 0 0.042 rpy=0 0 0 -> xyz=-0.025 0 0.042 rpy=0 0 0

Commit message: Configure urdf gripper friction

File: src/maniskill_elirobots/assets/ec63/ec63_description.urdf (robot description, URDF)
Before this commit: robot ec63, 13 links, 12 joints
Joints:
- joint finger_1_joint: limit lower=0 upper=0.02 effort=10 velocity=0.1 -> lower=0 upper=0.02 effort=100 velocity=0.2
- joint finger_2_joint: limit lower=0 upper=0.02 effort=10 velocity=0.1 -> lower=0 upper=0.02 effort=100 velocity=0.2; mimic (none) -> joint=finger_1_joint
